File: porta-jelly.kicad_pcb (KiCad board)
At the start: 2 copper layers, 50 x 77.5 mm, 40 parts, among them J1 USB_B_Micro, J10 8, J11 BATT-, J2 BATT+, J3 1, J4 2, J5 3, J6 4, J7 5, J8 6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

Commit message: Revised board design
Parts:
- L1: footprint Inductor_SMD:L_Coilcraft_XxL4040 -> porta-jelly:LQH44PH1R0MPRL
- Q1: value Q_PMOS_GDS -> DMP3099L
- SW1: value SW_SPST -> PWR; footprint Connector_PinHeader_2.54mm:PinHeader_1x02_P2.54mm_Vertical -> porta-jelly:SK12D07VG5
- U3: footprint Package_SO:SOIC-8-1EP_3.9x4.9mm_P1.27mm_EP2.29x3mm_ThermalVias -> porta-jelly:SOIC-8-1EP_3.9x4.9mm_P1.27mm_EP2.29x3mm_ThermalVias
- moved FID1 66.1 mm to (95.0, 132.5)
- moved SW1 42.0 mm to (132.0, 82.0), turned to 90 degrees
- moved FID3 40.0 mm to (125.0, 132.5)
- moved FID2 37.8 mm to (110.0, 91.0)
- moved U1 35.0 mm to (92.8, 83.0)
- moved C1 32.4 mm to (89.0, 78.5), turned to 0 degrees
- moved R4 12.5 mm to (127.8, 82.0)
- moved Q1 8.70 mm to (124.9, 82.0), turned to 180 degrees
- moved C3 7.11 mm to (118.5, 77.5), turned to -90 degrees
- moved C5 6.52 mm to (114.5, 77.5), turned to -90 degrees
- moved C4 5.52 mm to (116.5, 77.5), turned to -90 degrees
- moved C2 5.22 mm to (114.8, 72.0)
- moved R2 5.22 mm to (116.2, 72.0)
- moved D5 5.00 mm to (108.1, 67.0)
- moved D2 5.00 mm to (102.0, 67.0)
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Connections:
- SW1 pad 1: GND -> Net-(Q1-G)
- SW1 pad 2: Net-(Q1-G) -> GND
- U2 pad 1: /DATA -> unconnected-(U2-GPIO0-Pad1)
- U2 pad 13: unconnected-(U2-GND-Pad13) -> GND
- U2 pad 2: /CLOCK -> unconnected-(U2-GPIO1-Pad2)
- U2 pad 21: unconnected-(U2-GPIO16-Pad21) -> /DATA
- U2 pad 22: unconnected-(U2-GPIO17-Pad22) -> /LATCH
- U2 pad 24: unconnected-(U2-GPIO18-Pad24) -> /CLOCK
- U2 pad 28: unconnected-(U2-GND-Pad28) -> GND
- U2 pad 3: unconnected-(U2-GND-Pad3) -> GND
- U2 pad 4: /LATCH -> unconnected-(U2-GPIO2-Pad4)
- U2 pad 42: unconnected-(U2-GND-Pad42) -> GND
- U2 pad 8: unconnected-(U2-GND-Pad8) -> GND
Routing:
- net Net-(J7-Pin_2): track 0.00 -> 71.6 mm
- net Net-(J8-Pin_2): track 0.00 -> 60.8 mm
- net Net-(J9-Pin_2): track 0.00 -> 49.9 mm
- net Net-(J10-Pin_2): track 0.00 -> 43.7 mm
- net GND: track 1.01 -> 23.9 mm, vias 1 -> 15
- net Net-(J3-Pin_2): track 40.9 -> 18.7 mm
- net /CLOCK: track 0.00 -> 21.8 mm
- net /LATCH: track 0.00 -> 17.2 mm
- net Net-(J4-Pin_2): track 40.1 -> 23.1 mm
- net +5V: track 169.3 -> 186.2 mm
- net /DATA: track 0.00 -> 15.0 mm
- net Net-(J6-Pin_2): track 56.5 -> 42.9 mm
- net Net-(J5-Pin_2): track 46.1 -> 33.0 mm
- net unconnected-(J1-Shield-Pad6): track 0.00 -> 12.7 mm
- net Net-(Q1-G): track 1.67 -> 6.66 mm
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- added copper zone on F.Cu, net +5V
- added copper zone on F.Cu, net Net-(Q1-S)
Other:
- board size 50 x 77.5 mm -> 50 x 72.5 mm

Commit message: Final board, schematic updates, LCSC order codes
Routing:
- net +5V: track 186.2 -> 188.0 mm
Other:
- board text added: "Porta Jelly ghub:HarkonenBade/porta-jelly Harkonen 2023-03-15"
