File: porta-jelly.kicad_sch (KiCad schematic)
At the start: 40 parts, among them J1 USB_B_Micro, J10 8, J11 BATT-, J2 BATT+, J3 1, J4 2, J5 3, J6 4, J7 5, J8 6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

Commit message: Revised board design
Parts:
- C1: symbol Device:C -> Device:C_Small
- L1: footprint Inductor_SMD:L_Coilcraft_XxL4040 -> porta-jelly:LQH44PH1R0MPRL; LCSC (none) -> C1857967
- SW1: value SW_SPST -> PWR; footprint Connector_PinHeader_2.54mm:PinHeader_1x02_P2.54mm_Vertical -> porta-jelly:SK12D07VG5; symbol Switch:SW_SPST -> Switch:SW_SPDT; LCSC (none) -> C3020419
- U3: footprint Package_SO:SOIC-8-1EP_3.9x4.9mm_P1.27mm_EP2.29x3mm_ThermalVias -> porta-jelly:SOIC-8-1EP_3.9x4.9mm_P1.27mm_EP2.29x3mm_ThermalVias; LCSC (none) -> C181692
Connections:
- net CLOCK: now also U2.24 (GPIO18); no longer U2.2 (GPIO1)
- net DATA: now also U2.21 (GPIO16); no longer U2.1 (GPIO0)
- net GND: now also SW1.2 (B), U2.13 (GND), U2.28 (GND), U2.3 (GND), U2.42 (GND), U2.8 (GND); no longer SW1.1 (A)
- net LATCH: now also U2.22 (GPIO17); no longer U2.4 (GPIO2)
- net at Q1.1 (G), R4.1: now also SW1.1 (A); no longer SW1.2 (B)
- no-connect marks 42 -> 37
Other:
- moved on the sheet: C1

Commit message: Final board, schematic updates, LCSC order codes
Parts:
- C2, C6, C7, C8: LCSC (none) -> C19702
- C3, C4, C5: LCSC (none) -> C159801
- D1: LCSC (none) -> C146335
- D2, D3, D4, D5: LCSC (none) -> C497961
- J1: LCSC (none) -> C136000
- Q1: LCSC (none) -> C155244
- R2, R3: LCSC (none) -> C307263
- U1: LCSC (none) -> C5947
Changed lines of the file:
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@@
+      (effects (font (size 1.27 1.27)) hide)
+    )
+    (property "LCSC" "C19702" (at 158.75 132.08 0)
       (effects (font (size 1.27 1.27)) hide)
     )
@@
       (effects (font (size 1.27 1.27)) hide)
     )
+    (property "LCSC" "C497961" (at 95.25 132.08 0)
+      (effects (font (size 1.27 1.27)) hide)
+    )
     (pin "1")
     (pin "2")
@@
       (effects (font (size 1.27 1.27)) hide)
     )
+    (property "LCSC" "C159801" (at 143.51 115.57 0)
+      (effects (font (size 1.27 1.27)) hide)
+    )
     (pin "1")
     (pin "2")
@@
       (effects (font (size 1.27 1.27)) hide)
     )
+    (property "LCSC" "C497961" (at 86.36 132.08 0)
+      (effects (font (size 1.27 1.27)) hide)
+    )
     (pin "1")
     (pin "2")
@@
     )
     (property "Datasheet" "http://www.ti.com/lit/ds/symlink/sn74hc595.pdf" (at 224.79 53.34 0)
+      (effects (font (size 1.27 1.27)) hide)
+    )
+    (property "LCSC" "C5947" (at 224.79 53.34 0)
       (effects (font (size 1.27 1.27)) hide)
     )
@@
       (effects (font (size 1.27 1.27)) hide)
     )
+    (property "LCSC" "C155244" (at 182.88 115.57 0)
+      (effects (font (size 1.27 1.27)) hide)
+    )
     (pin "1")
     (pin "2")
@@
     )
     (property "Datasheet" "~" (at 158.75 127 0)
+      (effects (font (size 1.27 1.27)) hide)
+    )
+    (property "LCSC" "C307263" (at 158.75 127 0)
       (effects (font (size 1.27 1.27)) hide)
     )
@@
       (effects (font (size 1.27 1.27)) hide)
     )
+    (property "LCSC" "C159801" (at 152.4 115.57 0)
+      (effects (font (size 1.27 1.27)) hide)
+    )
     (pin "1")
     (pin "2")
@@
       (effects (font (size 1.27 1.27)) hide)
     )
+    (property "LCSC" "C19702" (at 107.95 115.57 0)
+      (effects (font (size 1.27 1.27)) hide)
+    )
     (pin "1")
     (pin "2")
@@
       (effects (font (size 1.27 1.27)) hide)
     )
+    (property "LCSC" "C146335" (at 158.75 31.75 0)
+      (effects (font (size 1.27 1.27)) hide)
+    )
     (pin "1")
     (pin "2")
@@
     )
     (property "Datasheet" "~" (at 81.28 120.65 0)
+      (effects (font (size 1.27 1.27)) hide)
+    )
+    (property "LCSC" "C19702" (at 81.28 120.65 0)
       (effects (font (size 1.27 1.27)) hide)
     )
@@
       (effects (font (size 1.27 1.27)) hide)
     )
+    (property "LCSC" "C497961" (at 78.74 132.08 0)
+      (effects (font (size 1.27 1.27)) hide)
+    )
     (pin "1")
     (pin "2")
@@
       (effects (font (size 1.27 1.27)) hide)
     )
+    (property "LCSC" "C497961" (at 102.87 132.08 0)
+      (effects (font (size 1.27 1.27)) hide)
+    )
     (pin "1")
     (pin "2")
@@
       (effects (font (size 1.27 1.27)) hide)
     )
+    (property "LCSC" "C159801" (at 161.29 115.57 0)
+      (effects (font (size 1.27 1.27)) hide)
+    )
     (pin "1")
     (pin "2")
@@
     )
     (property "Datasheet" "~" (at 71.12 119.38 0)
+      (effects (font (size 1.27 1.27)) hide)
+    )
+    (property "LCSC" "C136000" (at 67.31 118.11 0)
       (effects (font (size 1.27 1.27)) hide)
     )
@@
       (effects (font (size 1.27 1.27)) hide)
     )
+    (property "LCSC" "C19702" (at 151.13 127 0)
+      (effects (font (size 1.27 1.27)) hide)
+    )
     (pin "1")
     (pin "2")
@@
       (effects (font (size 1.27 1.27)) hide)
     )
+    (property "LCSC" "C307263" (at 81.28 115.57 0)
+      (effects (font (size 1.27 1.27)) hide)
+    )
